File: hardware/solo-fpc1020/solo-fp1020.brd (EAGLE design)
At the start: 26 x 16 mm, 27 parts, among them J1 USB1061-XX-X-X_REVA

Commit message: v1
Parts:
- moved GND1 21.4 mm to (24.5, 2.50)
- moved 3V1 3.20 mm to (24.5, 4.50)
- moved SWCLK1 2.83 mm to (24.5, 8.50)
- moved SWDIO1 2.83 mm to (24.5, 10.5)
- moved STX->1 2.50 mm to (24.5, 6.50)
- turned C4 to 0 degrees
- turned C5 to 0 degrees
- turned C8 to 0 degrees
- turned C9 to 0 degrees
Connections:
- removed net AMS_IRQ: ST2.3
Routing:
- net +3V3: track 0.00 -> 47.5 mm, vias 0 -> 2
- net +5V: track 0.00 -> 25.9 mm, vias 0 -> 2
- net N$14: track 0.00 -> 17.9 mm, vias 0 -> 1
- net D+: track 0.00 -> 17.2 mm, vias 0 -> 2
- net D-: track 0.00 -> 16.0 mm, vias 0 -> 2
- net N$10: track 0.00 -> 14.5 mm, vias 0 -> 1
- net N$13: track 0.00 -> 11.7 mm, vias 0 -> 1
- net N$1: track 0.00 -> 11.5 mm, vias 0 -> 1
- net GND: track 0.00 -> 9.97 mm, vias 0 -> 7
- net CS_N: track 0.00 -> 8.85 mm, vias 0 -> 2
- net SPICLK: track 0.00 -> 7.95 mm, vias 0 -> 2
- net RST: track 0.00 -> 7.70 mm, vias 0 -> 2
- net IRQ: track 0.00 -> 7.43 mm, vias 0 -> 2
- net +1V8: track 0.00 -> 7.37 mm
- net SWDIO: track 0.00 -> 5.67 mm, vias 0 -> 1
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Other:
- outline, holes or cut-outs redrawn

Commit message: .
Parts:
- removed C11: .1u, efm-fido:C0402
- removed C3, C7, C8, C9: 4.7u, efm-fido:C0402
- removed L1: RGB_LED_1X1CL-505S-X-SD-T, efm-fido:CL-505S-X-SD-T
- removed L2: NCP114AMX180TCG, efm-fido:REG_NCP114AMX330TCG
- removed L3: NCP114AMX330TCG, efm-fido:REG_NCP114AMX330TCG
- added D1, D2: LTW-C191TLA, LTW-C191TLA:LEDC1608X65N
- added U1: AP2112K-3.3TRG1, AP2112K-3.3TRG1:SOT95P285X140-5N
- added U2: AP2112K-1.8TRG1, AP2112K-3.3TRG1:SOT95P285X140-5N
- C1, C10, C13, C2, C4, C5, C6: device efm-fido:C0402 -> rcl:C0603
- R1: device efm-fido:R0402 -> rcl:R0603
- moved 5V1 5.52 mm to (6.50, 2.00)
- moved C4 3.16 mm to (15.5, 13.5), turned to 90 degrees
- moved C10 2.69 mm to (11.5, 13.5)
- moved C2 2.24 mm to (7.00, 2.50)
- moved C5 2.24 mm to (13.5, 13.5), turned to 90 degrees
- moved ST2 1.80 mm to (19.5, 8.00)
- moved U$4 1.80 mm to (18.5, 13.5)
- moved C13 1.58 mm to (20.0, 2.50)
- moved 3V1 1.50 mm to (24.5, 6.00)
- moved GND1 1.50 mm to (24.5, 4.00)
- moved STX->1 1.50 mm to (24.5, 8.00)
- moved SWCLK1 1.50 mm to (24.5, 10.0)
- moved SWDIO1 1.50 mm to (24.5, 12.0)
- moved C1 1.41 mm to (9.00, 2.50)
- moved Z1 1.25 mm to (5.50, 9.00)
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Connections:
- removed net N$13: L1.P$1, ST2.9
- net +1V8: now also U2.5; no longer C11.2, L2.1
- net +3V3: now also U1.5; no longer C3.1, C7.1, C8.1, C9.1, L3.1
- net +5V: now also U1.1, U1.3, U2.1, U2.3; no longer L2.3, L2.4, L3.3, L3.4
- net GND: now also U1.2, U2.2; no longer C11.1, C3.2, C7.2, C8.2, C9.2, L2.2, L3.2
- net N$1: now also D1.A, D2.A; no longer L1.P$4
- net N$10: now also D2.C; no longer L1.P$2
- net N$14: now also D1.C; no longer L1.P$3
Routing:
- net N$13: track 11.7 -> 0.00 mm, vias 1 -> 0
- net N$1: track 11.5 -> 22.8 mm, vias 1 -> 2
- net N$10: track 14.5 -> 7.76 mm
- net N$14: track 17.9 -> 12.7 mm
- net +3V3: track 47.5 -> 52.5 mm, vias 2 -> 3
- net D-: track 16.0 -> 21.0 mm
- net IRQ: track 7.43 -> 11.3 mm
- net GND: track 9.97 -> 6.15 mm, vias 7 -> 4
- net D+: track 17.2 -> 20.4 mm
- net MOSI: track 4.32 -> 5.90 mm, vias 0 -> 2
- net SPICLK: track 7.95 -> 9.49 mm, vias 2 -> 0
- net RST: track 7.70 -> 9.05 mm
- net +5V: track 25.9 -> 27.1 mm, vias 2 -> 1
- net SWCLK: track 4.48 -> 3.39 mm
- net STX->: track 3.75 -> 2.75 mm
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