File: hardware/solo-fpc1020/solo-fp1020.sch (EAGLE design)
At the start: 27 parts, among them J1 USB1061-XX-X-X_REVA

Commit message: v1
Connections:
- removed net AMS_IRQ: ST2.PC15
Changed lines of the file:
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@@
 </variantdefs>
 <classes>
-<class number="0" name="default" width="0.1524" drill="0.2032">
-<clearance class="0" value="0.1016"/>
+<class number="0" name="default" width="0.15" drill="0.2">
+<clearance class="0" value="0.1"/>
 </class>
-<class number="1" name="nfc" width="0.0889" drill="0.2032">
-<clearance class="1" value="0.0889"/>
+<class number="1" name="power" width="0.2" drill="0.2">
+<clearance class="1" value="0.15"/>
 </class>
 </classes>
@@
 </busses>
 <nets>
-<net name="+5V" class="0">
+<net name="+5V" class="1">
 <segment>
 <pinref part="P+5" gate="1" pin="+5V"/>
@@
 </segment>
 </net>
-<net name="GND" class="0">
+<net name="GND" class="1">
 <segment>
 <pinref part="SUPPLY3" gate="PE" pin="PE"/>
@@
 </segment>
 </net>
-<net name="+3V3" class="0">
+<net name="+3V3" class="1">
 <segment>
 <pinref part="+3V9" gate="G$1" pin="+3V3"/>
@@
 </segment>
 </net>
-<net name="AMS_IRQ" class="0">
-<segment>
-<pinref part="ST2" gate="G$1" pin="PC15"/>
-<wire x1="195.58" y1="99.06" x2="198.12" y2="99.06" width="0.1524" layer="91"/>
-<label x="198.12" y="99.06" size="1.778" layer="95"/>
-</segment>
-</net>
 <net name="MISO" class="0">
 <segment>
@@
 </segment>
 </net>
-<net name="+1V8" class="0">
+<net name="+1V8" class="1">
 <segment>
 <pinref part="U$1" gate="G$1" pin="VDD"/>

Commit message: .
Parts:
- removed C11: .1u, efm-fido:CAPACITOR
- removed C3, C7, C8, C9: 4.7u, efm-fido:CAPACITOR
- removed L1: RGB_LED_1X1CL-505S-X-SD-T, efm-fido:RGB_LED_1X1CL-505S-X-SD-T
- removed L2: NCP114AMX180TCG, efm-fido:NCP114AMX330TCG
- removed L3: NCP114AMX330TCG, efm-fido:NCP114AMX330TCG
- added D1, D2: LTW-C191TLA, LTW-C191TLA:LTW-C191TLA
- added U1: AP2112K-3.3TRG1, AP2112K-3.3TRG1:AP2112K-3.3TRG1
- added U2: AP2112K-1.8TRG1, AP2112K-3.3TRG1:AP2112K-3.3TRG1
- C1, C10, C13, C2, C4, C5, C6: device efm-fido:CAPACITOR -> rcl:C-EUC0603
- R1: device efm-fido:RESISTOR -> rcl:R-EU_R0603
Connections:
- removed net N$13: L1.CBLUE, ST2.PA3
- net +1V8: now also U2.VOUT; no longer C11.2, L2.OUT
- net +3V3: now also U1.VOUT; no longer C3.1, C7.1, C8.1, C9.1, L3.OUT
- net +5V: now also U1.EN, U1.VIN, U2.EN, U2.VIN; no longer L2.EN, L2.IN, L3.EN, L3.IN
- net GND: now also U1.GND, U2.GND; no longer C11.1, C3.2, C7.2, C8.2, C9.2, L2.GND, L3.GND
- net N$1: now also D1.A, D2.A; no longer L1.A2
- net N$10: now also D2.C; no longer L1.CRED
- net N$14: now also D1.C; no longer L1.CGREEN
Other:
- moved on the sheet: C1, C10, C2, R1
